File: Implementation/test-fixture/test-fixture.kicad_sch (KiCad schematic)
At the start: 2 parts, among them J1 Conn_02x31_Odd_Even, U1 TCA9555PWR

Commit message: First draft PCB for test fixture
Parts:
- removed U1: TCA9555PWR, Package_SO:TSSOP-24_4.4x7.8mm_P0.65mm, symbol Interface_Expansion:TCA9555PWR
- added A2: Clone_Mega2560_Pro_Socket, PCM_arduino-library:Clone_Mega2560_Pro_Socket, symbol PCM_arduino-library:Clone_Mega2560_Pro_Socket
- added DS1: WC1602A, Display:WC1602A, symbol Display_Character:WC1602A
- added R1, R2, R4: 10k, Resistor_THT:R_Axial_DIN0207_L6.3mm_D2.5mm_P10.16mm_Horizontal, symbol Device:R_US
- added R3: 220, Resistor_THT:R_Axial_DIN0207_L6.3mm_D2.5mm_P10.16mm_Horizontal, symbol Device:R_US
- added RV1: 10k, Potentiometer_THT:Potentiometer_ACP_CA9-V10_Vertical, symbol Device:R_Potentiometer_US
- added SW1, SW2: SW_Push, Button_Switch_THT:SW_PUSH_6mm, symbol Switch:SW_Push
- J1: footprint (none) -> Connector_Nandy:EDAC_395-062-520-350
Connections:
- net +5V: now also A2.5V1 (5V), A2.5V3 (5V), DS1.2 (VDD), R1.1, R2.1, R4.1, RV1.1
- net GND: now also J1.20 (Pin_20), A2.GND1 (GND), A2.GND2 (GND), DS1.1 (VSS), DS1.16 (LED(-)), DS1.5 (R/W), RV1.3, SW1.2, SW2.2
- net PL7: now reaches J1.10 (Pin_10)
- net PL7: now also A2.D42
- net PC0: now reaches J1.11 (Pin_11)
- net PC0: now also A2.D37
- net PC1: now reaches J1.12 (Pin_12)
- net PC1: now also A2.D36
- net PC2: now reaches J1.13 (Pin_13)
- net PC2: now also A2.D35
- net PC3: now reaches J1.14 (Pin_14)
- net PC3: now also A2.D34
- net PC4: now reaches J1.15 (Pin_15)
- net PC4: now also A2.D33
- net PC5: now reaches J1.16 (Pin_16)
- net PC5: now also A2.D32
- net PC6: now reaches J1.17 (Pin_17)
- net PC6: now also A2.D31
- net PC7: now reaches J1.18 (Pin_18)
- net PC7: now also A2.D30
- net D3: now reaches J1.19 (Pin_19)
- net D3: now also A2.D3 (D3_INT1)
- net PK0: now reaches J1.21 (Pin_21)
- net PK0: now also A2.A8
- net PK1: now reaches J1.22 (Pin_22)
- net PK1: now also A2.A9
- net PK2: now reaches J1.23 (Pin_23)
- net PK2: now also A2.A10
- net PK3: now reaches J1.24 (Pin_24)
- net PK3: now also A2.A11
- net PK4: now reaches J1.25 (Pin_25)
- net PK4: now also A2.A12
- net PK5: now reaches J1.26 (Pin_26)
- net PK5: now also A2.A13
- net PK6: now reaches J1.27 (Pin_27)
- net PK6: now also A2.A14
- net PK7: now reaches J1.28 (Pin_28)
- net PK7: now also A2.A15
- net D4: now reaches J1.29 (Pin_29)
- net D4: now also A2.D4
- net PL0: now reaches J1.3 (Pin_3)
- net PL0: now also A2.D49
- net D5: now reaches J1.30 (Pin_30)
- net D5: now also A2.D5
- net PA0: now reaches J1.33 (Pin_33)
- net PA0: now also A2.D22
- net PA1: now reaches J1.34 (Pin_34)
- net PA1: now also A2.D23
- net PA2: now reaches J1.35 (Pin_35)
- net PA2: now also A2.D24
- net PA3: now reaches J1.36 (Pin_36)
- net PA3: now also A2.D25
- net PA4: now reaches J1.37 (Pin_37)
- net PA4: now also A2.D26
- net PA5: now reaches J1.38 (Pin_38)
- net PA5: now also A2.D27
- net PA6: now reaches J1.39 (Pin_39)
- net PA6: now also A2.D28
- net PL1: now reaches J1.4 (Pin_4)
- net PL1: now also A2.D48
- net PA7: now reaches J1.40 (Pin_40)
- net PA7: now also A2.D29
- net PF0: now reaches J1.41 (Pin_41)
- net PF0: now also A2.A0
- net PF1: now reaches J1.42 (Pin_42)
- net PF1: now also A2.A1
- net PF2: now reaches J1.43 (Pin_43)
- net PF2: now also A2.A2
- net PF3: now reaches J1.44 (Pin_44)
- net PF3: now also A2.A3
- net PF4: now reaches J1.45 (Pin_45)
- net PF4: now also A2.A4
- net PF5: now reaches J1.46 (Pin_46)
- net PF5: now also A2.A5
- net PF6: now reaches J1.47 (Pin_47)
- net PF6: now also A2.A6
- net PF7: now reaches J1.48 (Pin_48)
- net PF7: now also A2.A7
- net D6: now reaches J1.49 (Pin_49)
- net D6: now also A2.D6
- net PL2: now reaches J1.5 (Pin_5)
- net PL2: now also A2.D47
- net GND_DET: now reaches J1.50 (Pin_50)
- net GND_DET: now also A2.D8, R4.2
- net D2: now reaches J1.51 (Pin_51)
- net D2: now also A2.D2 (D2_INT0)
- net D7: now reaches J1.52 (Pin_52)
- net D7: now also A2.D7
- net PB0: now reaches J1.53 (Pin_53)
- net PB0: now also A2.D53 (D53_CS)
- net PB1: now reaches J1.54 (Pin_54)
- net PB1: now also A2.D52 (D52_SCK)
- net PB2: now reaches J1.55 (Pin_55)
- net PB2: now also A2.D51 (D51_MOSI)
- net PB3: now reaches J1.56 (Pin_56)
- net PB3: now also A2.D50 (D50_MISO)
- net PB4: now reaches J1.57 (Pin_57)
- net PB4: now also A2.D10
- net PB5: now reaches J1.58 (Pin_58)
- net PB5: now also A2.D11
- net PB6: now reaches J1.59 (Pin_59)
- net PB6: now also A2.D12
- net PL3: now reaches J1.6 (Pin_6)
- net PL3: now also A2.D46
- net PB7: now reaches J1.60 (Pin_60)
- net PB7: now also A2.D13
- net PL4: now reaches J1.7 (Pin_7)
- net PL4: now also A2.D45
- net PL5: now reaches J1.8 (Pin_8)
- net PL5: now also A2.D44
- net PL6: now reaches J1.9 (Pin_9)
- net PL6: now also A2.D43
- new net: DS1.3 (VO), RV1.2
- new net: DS1.15 (LED(+)), R3.1
- new net LCD_BL: A2.D9, R3.2
- new net LCD_D4: A2.D14 (D14/TX3), DS1.11 (D4)
- new net LCD_D5: A2.D15 (D15/RX3), DS1.12 (D5)
- new net LCD_D6: A2.D16 (D16/TX2), DS1.13 (D6)
- new net LCD_D7: A2.D17 (D17/RX2), DS1.14 (D7)
- new net LCD_E: A2.D39, DS1.6 (E)
- new net LCD_RS: A2.D38, DS1.4 (RS)
- new net SW1: A2.D41, R2.2, SW1.1
- new net SW2: A2.D40, R1.2, SW2.1
- no-connect marks 0 -> 4
Other:
- moved on the sheet: J1
